File: Telephone_Line_Card.kicad_pcb (KiCad board)
At the start: 2 copper layers, 101.6 x 63.5 mm, 0 parts

Commit message: some pcb changes
Parts:
- added C1: 100uF, Capacitor_THT:CP_Radial_D8.0mm_P5.00mm, F.Cu at (26.4, 5.08)
- added C2: 100uF/100V, Capacitor_THT:CP_Radial_D12.5mm_P5.00mm, F.Cu at (17.0, 36.6)
- added C3: 0.1uF, Capacitor_THT:C_Disc_D4.7mm_W2.5mm_P5.00mm, F.Cu at (32.8, 30.0)
- added C4: 2uF/100V, Capacitor_THT:C_Rect_L18.0mm_W8.0mm_P15.00mm_FKS3_FKP3, F.Cu at (58.4, 56.6)
- added C5: 2uF/100V, Capacitor_THT:C_Rect_L18.0mm_W8.0mm_P15.00mm_FKS3_FKP3, F.Cu at (58.4, 48.0)
- added C6: RC .1uF/47R, Capacitor_THT:C_Rect_L24.0mm_W10.9mm_P22.50mm_MKT, F.Cu at (94.5, 45.7)
- added C7: 47uF/10V, Capacitor_THT:C_Radial_D10.0mm_H12.5mm_P5.00mm, F.Cu at (40.4, 73.4)
- added D1: OFFHOOK_LED, LED_THT:LED_D5.0mm, F.Cu at (91.7, 11.7)
- added D2: RING_LED, LED_THT:LED_D5.0mm, F.Cu at (91.7, 19.8)
- added D3: 1N4148, Diode_THT:D_DO-35_SOD27_P7.62mm_Horizontal, F.Cu at (78.0, 36.6)
- added D4: 1N4148, Diode_THT:D_DO-35_SOD27_P7.62mm_Horizontal, F.Cu at (17.5, 56.1)
- added D5: 1N4148, Diode_THT:D_DO-35_SOD27_P7.62mm_Horizontal, F.Cu at (20.1, 48.5)
- added D6: 1N4148, Diode_THT:D_DO-35_SOD27_P7.62mm_Horizontal, F.Cu at (52.3, 77.5)
- added H1: MountingHole, MountingHole:MountingHole_3.2mm_M3, F.Cu at (3.81, 3.81)
- added H2: MountingHole, MountingHole:MountingHole_3.2mm_M3, F.Cu at (97.8, 3.81)
- added H3: MountingHole, MountingHole:MountingHole_3.2mm_M3, F.Cu at (97.8, 85.1)
- added H4: MountingHole, MountingHole:MountingHole_3.2mm_M3, F.Cu at (3.81, 85.1)
- added J1: Conn_01x12, Connector_PinSocket_2.54mm:PinSocket_1x12_P2.54mm_Horizontal, F.Cu at (10.7, 12.7)
- added J2: RJ11, TerminalBlock:TerminalBlock_bornier-2_P5.08mm, F.Cu at (94.5, 39.1)
- added K1: TELTONE_M949-1, Teltone_M949_Line_Sense_Relay:Teltone_M-949-1, F.Cu at (66.3, 65.0)
- added K2: G5V-2, Relay_THT:Relay_DPDT_Omron_G5V-2, F.Cu at (78.0, 40.9)
- added Q1: 2N3904, Package_TO_SOT_THT:TO-92_Wide, F.Cu at (74.7, 26.2)
- added R1: 330R/2W, Resistor_THT:R_Axial_DIN0617_L17.0mm_D6.0mm_P30.48mm_Horizontal, F.Cu at (58.4, 65.0)
- added R10: 5K, Resistor_THT:R_Axial_DIN0309_L9.0mm_D3.2mm_P12.70mm_Horizontal, F.Cu at (47.2, 73.7)
- added R11: 10K, Resistor_THT:R_Axial_DIN0309_L9.0mm_D3.2mm_P12.70mm_Horizontal, F.Cu at (49.8, 15.2)
- added R2: 330R/2W, Resistor_THT:R_Axial_DIN0617_L17.0mm_D6.0mm_P30.48mm_Horizontal, F.Cu at (58.4, 39.6)
- added R3: 1K, Resistor_THT:R_Axial_DIN0309_L9.0mm_D3.2mm_P12.70mm_Horizontal, F.Cu at (77.2, 11.4)
- added R4: 1K, Resistor_THT:R_Axial_DIN0309_L9.0mm_D3.2mm_P12.70mm_Horizontal, F.Cu at (85.6, 19.8)
- added R5: 1K, Resistor_THT:R_Axial_DIN0309_L9.0mm_D3.2mm_P12.70mm_Horizontal, F.Cu at (77.2, 19.1)
- added R6: 10K, Resistor_THT:R_Axial_DIN0309_L9.0mm_D3.2mm_P12.70mm_Horizontal, F.Cu at (64.5, 15.2)
- added R7: 10K, Resistor_THT:R_Axial_DIN0309_L9.0mm_D3.2mm_P12.70mm_Horizontal, F.Cu at (49.8, 11.4)
- added R8: 620R, Resistor_THT:R_Axial_DIN0309_L9.0mm_D3.2mm_P12.70mm_Horizontal, F.Cu at (75.2, 77.5)
- added R9: 5K, Resistor_THT:R_Axial_DIN0309_L9.0mm_D3.2mm_P12.70mm_Horizontal, F.Cu at (62.5, 73.7)
- added T1: 600:600, Transformer_Bourns_LM-NP-100x_Signal_Transformers:Transformer_Bourns_LM-NP-1001_1xSec, F.Cu at (37.3, 48.5)
- added TH1: Thermistor_PTC, Fuse:Fuse_Bourns_MF-RG400, F.Cu at (85.6, 64.0)
- added U1: 4N35, Package_DIP:DIP-6_W7.62mm, F.Cu at (27.9, 78.0)
Routing:
- net +5V: track 0.00 -> 190.9 mm
- net RING_BUS(T): track 0.00 -> 141.1 mm
- net RT: track 0.00 -> 103.2 mm
- net RING_BUS(R): track 0.00 -> 91.9 mm
- net SHK: track 0.00 -> 91.4 mm
- net GND: track 0.00 -> 78.0 mm
- net RM: track 0.00 -> 59.3 mm, vias 0 -> 2
- net Net-(C6-Pad2): track 0.00 -> 55.0 mm
- net VOICE_LINE(R): track 0.00 -> 52.1 mm
- net Earth: track 0.00 -> 47.0 mm
- net Net-(C5-Pad1): track 0.00 -> 39.2 mm
- net Net-(C3-Pad1): track 0.00 -> 36.6 mm
- net Net-(C4-Pad1): track 0.00 -> 30.5 mm
- net Net-(D6-Pad1): track 0.00 -> 28.4 mm
- net Net-(C6-Pad1): track 0.00 -> 25.5 mm
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- added copper zone on F.Cu, net GND
Other:
- board size 101.6 x 63.5 mm -> 101.6 x 88.9 mm
- net class Default: clearance 0.2 -> 0.2032; trace_width 0.25 -> 0.762; via_dia 0.8 -> 1.524; via_drill 0.4 -> 0.762
- rule trace_clearance: 0.2 -> 0.2032

Commit message: some more pcb changes
Parts:
- moved D6 110.6 mm to (141.5, 143.0)
- moved R10 110.6 mm to (136.4, 139.2)
- moved R8 110.6 mm to (164.3, 143.0)
- moved R9 110.6 mm to (151.6, 139.2)
- moved U1 110.6 mm to (117.1, 143.5)
- moved C7 110.6 mm to (129.5, 138.9)
- moved R3 109.2 mm to (166.1, 74.9)
- moved C1 109.2 mm to (115.3, 68.6)
- moved C2 109.2 mm to (105.9, 100.1)
- moved C6 109.2 mm to (183.4, 109.2)
- moved D4 109.2 mm to (106.4, 119.6)
- moved J1 109.2 mm to (99.6, 76.2)
- moved J2 109.2 mm to (183.4, 102.6)
- moved K2 109.2 mm to (166.9, 104.4)
- moved Q1 109.2 mm to (163.6, 89.7)
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Routing:
- net Net-(C3-Pad1): track 36.6 -> 46.0 mm
- net RING_BUS(T): track 141.1 -> 148.9 mm
- net GND: track 78.0 -> 84.7 mm
- net RING_BUS(R): track 91.9 -> 97.2 mm
- net VOICE_LINE(T): track 24.0 -> 19.2 mm
- net VOICE_LINE(R): track 52.1 -> 54.6 mm
- net Earth: track 47.0 -> 49.4 mm
- net RT: track 103.2 -> 105.1 mm
- net +5V: track 190.9 -> 189.7 mm
- net RM: track 59.3 -> 58.2 mm
- net Net-(D3-Pad2): track 18.5 -> 19.2 mm
- net Net-(R8-Pad1): track 14.9 -> 15.5 mm
Other:
- board text added: "+5V"
- board text added: "+VBAT/E"
- board text added: "-VBAT"
- board text added: "GND"
- board text added: "OFF-HOOK"
- board text added: "R"
- board text added: "RING"
- board text added: "RINGBUS(R)"
- board text added: "RINGBUS(T)"
- board text added: "RM"
- board text added: "RT"
- board text added: "SHK"
- board text added: "T"
- board text added: "TELECOM LINE CARD DMA, REV. A"
- board text added: "VOICE(R)"
- board text added: "VOICE(T)"

Commit message: generated gerbers
Routing:
- net SHK: track 91.4 -> 87.6 mm
